File: 6N2P_amp.kicad_pcb (KiCad board)
At the start: 2 copper layers, 225 x 100 mm, 78 parts, among them J1 guitar_in, J2 speaker, J3 fx_send, J4 fx_return, U1 ECC83, U2 ECC83, U3 6N1P, U4 DSN-MINI-360, U5 DSN-MINI-360, U6 DSN-MINI-360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

Commit message: snap
Parts:
- moved C13 355.3 mm to (221.0, 180.0)
- moved C12 347.8 mm to (205.0, 180.0)
- moved D3 343.4 mm to (146.0, -76.0)
- moved C11 335.7 mm to (202.0, 162.0)
- moved C16 312.2 mm to (217.0, 251.0)
- moved R13 301.6 mm to (24.0, 32.0)
- moved D4 301.3 mm to (146.0, -34.0)
- moved R20 292.1 mm to (194.0, 241.0)
- moved C15 290.5 mm to (196.0, 250.0)
- moved C14 287.6 mm to (205.0, 233.0)
- moved R22 286.5 mm to (220.0, 235.0)
- moved R17 241.8 mm to (203.0, 171.0)
- moved R21 206.5 mm to (222.0, 162.0)
- moved D5 134.3 mm to (223.0, 173.0)
- moved D6 76.0 mm to (212.0, 243.0)
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Routing:
- net GND: track 295.6 -> 310.6 mm
Changed lines of the file:
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@@
     (thickness 1.6)
     (drawings 11)
-    (tracks 198)
+    (tracks 199)
     (zones 0)
     (modules 78)
@@
   )
   (module Capacitor_THT:C_Rect_L9.0mm_W4.0mm_P7.50mm_MKT (layer F.Cu)
-    (at 16.625001 -117.894999)
+    (at 202 162)
     (descr "C, Rect series, Radial, pin pitch=7.50mm, , length*width=9*4.0mm^2, Capacitor, https://en.tdk.eu/inf/20/20/db/fc_2009/MKT_B32560_564.pdf")
     (tags "C Rect series Radial pin pitch 7.50mm  length 9mm width 4.0mm Capacitor")
@@
   )
   (module Capacitor_THT:C_Rect_L9.0mm_W4.0mm_P7.50mm_MKT (layer F.Cu)
-    (at 16.625001 -112.344999)
+    (at 205 180)
     (descr "C, Rect series, Radial, pin pitch=7.50mm, , length*width=9*4.0mm^2, Capacitor, https://en.tdk.eu/inf/20/20/db/fc_2009/MKT_B32560_564.pdf")
     (tags "C Rect series Radial pin pitch 7.50mm  length 9mm width 4.0mm Capacitor")
@@
   )
   (module Capacitor_THT:C_Rect_L9.0mm_W4.0mm_P7.50mm_MKT (layer F.Cu)
-    (at 27.275001 -117.894999)
+    (at 221 180)
     (descr "C, Rect series, Radial, pin pitch=7.50mm, , length*width=9*4.0mm^2, Capacitor, https://en.tdk.eu/inf/20/20/db/fc_2009/MKT_B32560_564.pdf")
     (tags "C Rect series Radial pin pitch 7.50mm  length 9mm width 4.0mm Capacitor")
@@
   )
   (module Resistor_THT:R_Axial_DIN0207_L6.3mm_D2.5mm_P10.16mm_Horizontal (layer F.Cu)
-    (at 309.685001 -64.754999)
+    (at 24 32)
     (descr "Resistor, Axial_DIN0207 series, Axial, Horizontal, pin pitch=10.16mm, 0.25W = 1/4W, length*diameter=6.3*2.5mm^2, http://cdn-reichelt.de/documents/datenblatt/B400/1_4W%23YAG.pdf")
     (tags "Resistor Axial_DIN0207 series Axial Horizontal pin pitch 10.16mm 0.25W = 1/4W length 6.3mm diameter 2.5mm")
@@
   )
   (module Resistor_THT:R_Axial_DIN0207_L6.3mm_D2.5mm_P10.16mm_Horizontal (layer F.Cu)
-    (at 270.565001 -61.184999)
+    (at 203 171)
     (descr "Resistor, Axial_DIN0207 series, Axial, Horizontal, pin pitch=10.16mm, 0.25W = 1/4W, length*diameter=6.3*2.5mm^2, http://cdn-reichelt.de/documents/datenblatt/B400/1_4W%23YAG.pdf")
     (tags "Resistor Axial_DIN0207 series Axial Horizontal pin pitch 10.16mm 0.25W = 1/4W length 6.3mm diameter 2.5mm")
@@
   )
   (module Capacitor_THT:C_Rect_L9.0mm_W4.0mm_P7.50mm_MKT (layer F.Cu)
-    (at 183.615001 -53.814999)
+    (at 205 233)
     (descr "C, Rect series, Radial, pin pitch=7.50mm, , length*width=9*4.0mm^2, Capacitor, https://en.tdk.eu/inf/20/20/db/fc_2009/MKT_B32560_564.pdf")
     (tags "C Rect series Radial pin pitch 7.50mm  length 9mm width 4.0mm Capacitor")
@@
   )
   (module Capacitor_THT:C_Rect_L9.0mm_W4.0mm_P7.50mm_MKT (layer F.Cu)
-    (at 169.105001 -39.264999)
+    (at 196 250)
     (descr "C, Rect series, Radial, pin pitch=7.50mm, , length*width=9*4.0mm^2, Capacitor, https://en.tdk.eu/inf/20/20/db/fc_2009/MKT_B32560_564.pdf")
     (tags "C Rect series Radial pin pitch 7.50mm  length 9mm width 4.0mm Capacitor")
@@
   )
   (module Capacitor_THT:C_Rect_L9.0mm_W4.0mm_P7.50mm_MKT (layer F.Cu)
-    (at 183.615001 -59.364999)
+    (at 217 251)
     (descr "C, Rect series, Radial, pin pitch=7.50mm, , length*width=9*4.0mm^2, Capacitor, https://en.tdk.eu/inf/20/20/db/fc_2009/MKT_B32560_564.pdf")
     (tags "C Rect series Radial pin pitch 7.50mm  length 9mm width 4.0mm Capacitor")
@@
   )
   (module Resistor_THT:R_Axial_DIN0207_L6.3mm_D2.5mm_P10.16mm_Horizontal (layer F.Cu)
-    (at 70.925001 -23.874999)
+    (at 194 241)
     (descr "Resistor, Axial_DIN0207 series, Axial, Horizontal, pin pitch=10.16mm, 0.25W = 1/4W, length*diameter=6.3*2.5mm^2, http://cdn-reichelt.de/documents/datenblatt/B400/1_4W%23YAG.pdf")
     (tags "Resistor Axial_DIN0207 series Axial Horizontal pin pitch 10.16mm 0.25W = 1/4W length 6.3mm diameter 2.5mm")
@@
   )
   (module OptoDevice:R_LDR_10x8.5mm_P7.6mm_Vertical (layer F.Cu)
-    (at 145.975001 -29.954999)
+    (at 222 162)
     (descr "Resistor, LDR 10x8.5mm")
     (tags "Resistor LDR10.8.5mm")
@@
   )
   (module OptoDevice:R_LDR_10x8.5mm_P7.6mm_Vertical (layer F.Cu)
-    (at 169.705001 -47.064999)
+    (at 220 235)
     (descr "Resistor, LDR 10x8.5mm")
     (tags "Resistor LDR10.8.5mm")
@@
   )
   (module OptoDevice:R_LDR_10x8.5mm_P7.6mm_Vertical (layer F.Cu)
-    (at 134.025001 -29.954999)
+    (at 134 -84)
     (descr "Resistor, LDR 10x8.5mm")
     (tags "Resistor LDR10.8.5mm")
@@
   )
   (module OptoDevice:R_LDR_10x8.5mm_P7.6mm_Vertical (layer F.Cu)
-    (at 172.265001 -57.114999)
+    (at 134 -42)
     (descr "Resistor, LDR 10x8.5mm")
     (tags "Resistor LDR10.8.5mm")
@@
   )
   (module LED_THT:LED_D5.0mm (layer F.Cu)
-    (at 135.475001 267.275001)
+    (at 146 -76)
     (descr "LED, diameter 5.0mm, 2 pins, http://cdn-reichelt.de/documents/datenblatt/A500/LL-504BC2E-009.pdf")
     (tags "LED diameter 5.0mm 2 pins")
@@
   )
   (module LED_THT:LED_D5.0mm (layer F.Cu)
-    (at 142.975001 267.275001)
+    (at 146 -34)
     (descr "LED, diameter 5.0mm, 2 pins, http://cdn-reichelt.de/documents/datenblatt/A500/LL-504BC2E-009.pdf")
     (tags "LED diameter 5.0mm 2 pins")
@@
   )
   (module LED_THT:LED_D5.0mm (layer F.Cu)
-    (at 135.475001 274.825001)
+    (at 223 173)
     (descr "LED, diameter 5.0mm, 2 pins, http://cdn-reichelt.de/documents/datenblatt/A500/LL-504BC2E-009.pdf")
     (tags "LED diameter 5.0mm 2 pins")
@@
   )
   (module LED_THT:LED_D5.0mm (layer F.Cu)
-    (at 142.975001 274.825001)
+    (at 212 243)
     (descr "LED, diameter 5.0mm, 2 pins, http://cdn-reichelt.de/documents/datenblatt/A500/LL-504BC2E-009.pdf")
     (tags "LED diameter 5.0mm 2 pins")
@@
   (segment (start 122.75 120.25) (end 127.5 120.25) (width 1) (layer B.Cu) (net 2))
   (segment (start 117 126) (end 122.75 120.25) (width 1) (layer B.Cu) (net 2))
+  (segment (start 127.5 120.25) (end 127.5 105.25) (width 1) (layer B.Cu) (net 2))
   (segment (start 34 117) (end 35 116) (width 1) (layer B.Cu) (net 5))
   (segment (start 30 117) (end 34 117) (width 1) (layer B.Cu) (net 5))

Commit message: introduced foot switch jack
Parts:
- added J5: foot_sw, micha_custom:Reichelt_EBS63P, F.Cu at (33.0, 71.0)
- moved R10 210.5 mm to (64.0, 82.0), turned to 270 degrees
- moved R11 206.8 mm to (53.0, 66.0), turned to 270 degrees
- moved R12 203.0 mm to (77.0, 66.0), turned to 270 degrees
- moved C14 103.4 mm to (102.0, 224.0), turned to 180 degrees
- moved C11 102.8 mm to (102.0, 186.0), turned to 180 degrees
- moved C7 100.3 mm to (76.0, 83.0), turned to 270 degrees
- moved R17 96.2 mm to (108.0, 186.0)
- moved C13 90.2 mm to (131.0, 186.0), turned to 180 degrees
- moved C16 90.1 mm to (131.0, 224.0), turned to 180 degrees
- moved R20 87.7 mm to (108.0, 224.0)
- moved R13 80.8 mm to (89.0, 80.0), turned to 270 degrees
- moved C6 78.9 mm to (52.0, 83.0), turned to 270 degrees
- moved C9 75.0 mm to (89.0, 67.0), turned to 270 degrees
- moved C12 59.3 mm to (146.0, 186.0), turned to 180 degrees
- moved C15 56.4 mm to (146.0, 224.0), turned to 180 degrees
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Routing:
- net /HV_A: track 0.00 -> 124.9 mm
- net GND: track 310.6 -> 393.4 mm
- net Net-(C11-Pad2): track 6.94 -> 75.1 mm
- net /HV_B: track 34.3 -> 83.2 mm
- net /HV_C: track 5.00 -> 50.5 mm
- net /fx_send: track 0.00 -> 43.1 mm
- net /HV_in: track 0.00 -> 38.9 mm
- net Net-(C15-Pad2): track 0.00 -> 21.9 mm
- net Net-(C12-Pad2): track 0.00 -> 21.9 mm
- net Net-(C3-Pad2): track 6.27 -> 23.1 mm
- net Net-(C15-Pad1): track 0.00 -> 15.0 mm
- net Net-(C12-Pad1): track 0.00 -> 15.0 mm
- net Net-(C16-Pad1): track 0.00 -> 12.9 mm
- net Net-(C13-Pad1): track 0.00 -> 12.9 mm
- net Net-(C14-Pad1): track 0.00 -> 12.1 mm
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