File: 6N2P_amp.kicad_pcb (KiCad board)
At the start: 2 copper layers, 225 x 100 mm, 79 parts, among them J1 guitar_in, J2 speaker, J3 fx_send, J4 fx_return, J5 foot_sw, U1 ECC83, U2 ECC83, U3 6N1P, U4 DSN-MINI-360, U5 DSN-MINI-360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

Commit message: genug fuer heute
Parts:
- moved R23 228.0 mm to (113.0, 143.0), turned to 90 degrees
- moved D3 221.2 mm to (103.0, 141.0), turned to 90 degrees
- moved R24 185.2 mm to (125.0, 143.0), turned to 90 degrees
- moved D4 175.3 mm to (135.0, 141.0), turned to 90 degrees
- moved R21 45.8 mm to (193.0, 197.4), turned to 270 degrees
- moved D5 35.5 mm to (204.0, 203.0), turned to 90 degrees
- moved R27 7.00 mm to (151.0, 113.0)
- moved R28 7.00 mm to (151.0, 130.0)
- moved R32 7.00 mm to (171.5, 102.0)
- moved R33 7.00 mm to (179.5, 106.0)
- moved U3 7.00 mm to (166.7, 116.8)
- moved U6 7.00 mm to (188.3, 116.8)
Routing:
- net /clean_channel_bypass: track 50.2 -> 103.9 mm
- net Net-(R23-Pad1): track 0.00 -> 42.0 mm
- net /od_A: track 7.93 -> 47.3 mm
- net GND: track 393.4 -> 385.3 mm
- net /power_anode: track 55.1 -> 48.1 mm

Commit message: LDRs
Parts:
- added D7: LED, LED_THT:LED_D5.0mm, F.Cu at (132.0, 127.0)
- added D8: LED, LED_THT:LED_D5.0mm, F.Cu at (132.0, 134.0)
- added R34: LDR03, OptoDevice:R_LDR_4.9x4.2mm_P2.54mm_Vertical, F.Cu at (123.0, 127.0)
- added R35: LDR03, OptoDevice:R_LDR_4.9x4.2mm_P2.54mm_Vertical, F.Cu at (123.0, 134.0)
- R18, R19, R21, R22, R23, R24: footprint OptoDevice:R_LDR_10x8.5mm_P7.6mm_Vertical -> OptoDevice:R_LDR_4.9x4.2mm_P2.54mm_Vertical
- moved R13 9.43 mm to (97.0, 85.0), turned to 180 degrees
- moved D1 6.32 mm to (57.0, 136.0)
- moved D2 4.70 mm to (85.0, 138.5)
- moved D4 3.00 mm to (132.0, 141.0)
- moved R23 3.00 mm to (113.0, 140.0)
- moved R24 2.83 mm to (123.0, 141.0)
- moved D3 2.24 mm to (105.0, 140.0)
Connections:
- C14 pad 2: Net-(C11-Pad2) -> Net-(C14-Pad2)
- R16 pad 1: Net-(C11-Pad2) -> Net-(R16-Pad1)
- R20 pad 1: Net-(C11-Pad2) -> Net-(C14-Pad2)
- U2 pad 3: Net-(C11-Pad2) -> Net-(R16-Pad1)
Routing:
- net Net-(R23-Pad1): track 42.0 -> 10.4 mm
- net Net-(R16-Pad1): track 0.00 -> 31.2 mm
- net GND: track 385.3 -> 407.9 mm
- net Net-(C11-Pad2): track 75.1 -> 68.1 mm
- net /HV_in: track 38.9 -> 32.8 mm
- net /clean_channel_bypass: track 103.9 -> 102.2 mm
- net /od_A: track 47.3 -> 48.1 mm

Commit message: snap
Parts:
- moved R15 20.4 mm to (108.0, 93.0), turned to 180 degrees
- moved U4 6.00 mm to (83.0, 107.0)
- moved U5 6.00 mm to (132.0, 107.0)
Routing:
- net /12V: track 0.00 -> 63.6 mm
- net /HV_B: track 83.2 -> 110.3 mm
- net GND: track 407.9 -> 418.4 mm
- net /od_A: track 48.1 -> 52.2 mm
- net /6.3V_U2: track 43.2 -> 39.1 mm

Commit message: snap
Parts:
- RV1, RV2, RV3, RV4, RV5, RV6: footprint Potentiometer_THT:Potentiometer_Alps_RK163_Single_Horizontal -> Connector_PinHeader_2.54mm:PinHeader_1x03_P2.54mm_Vertical
- moved R22 143.8 mm to (145.5, 112.0), turned to 180 degrees
- moved D6 141.0 mm to (143.0, 120.0)
- moved D5 118.0 mm to (143.0, 102.0), turned to 0 degrees
- moved R21 113.8 mm to (145.5, 94.0), turned to 180 degrees
- moved R32 17.7 mm to (189.0, 104.0), turned to 180 degrees
- moved U6 12.1 mm to (199.0, 111.0)
- moved R33 10.3 mm to (189.0, 110.0)
- moved C5 9.00 mm to (83.0, 120.0)
- moved D1 8.06 mm to (50.0, 132.0)
- moved R18 8.06 mm to (58.0, 132.0)
- moved R28 5.39 mm to (156.0, 128.0)
- moved U3 5.39 mm to (171.7, 114.8)
- moved R27 5.10 mm to (156.0, 114.0)
- moved C11 4.24 mm to (99.0, 189.0)
- moved C12 4.24 mm to (143.0, 189.0)
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Routing:
- net /fx_send: track 43.1 -> 82.1 mm
- net GND: track 418.4 -> 390.8 mm
- net Net-(C12-Pad1): track 15.0 -> 0.00 mm
- net Net-(C13-Pad1): track 12.9 -> 0.00 mm
- net Net-(C11-Pad1): track 12.1 -> 0.00 mm
- net Net-(R23-Pad1): track 10.4 -> 0.00 mm
- net /clean_channel_bypass: track 102.2 -> 111.9 mm
- net Net-(R32-Pad2): track 10.7 -> 19.4 mm
- net /6.3V_U3: track 33.4 -> 37.9 mm
- net /power_anode: track 48.1 -> 50.1 mm
- net Net-(C3-Pad1): track 25.1 -> 23.1 mm
- net Net-(C3-Pad2): track 23.1 -> 21.6 mm
- net /od_A: track 52.2 -> 50.7 mm
- net /power_gate: track 29.0 -> 29.7 mm
- net Net-(R16-Pad1): track 31.2 -> 31.9 mm

Commit message: more routing
Parts:
- moved RV11 85.4 mm to (187.0, 156.0)
- moved RV9 84.8 mm to (163.0, 156.0)
- moved RV10 84.2 mm to (139.0, 156.0)
- moved RV8 83.7 mm to (115.0, 156.0)
- moved C14 83.2 mm to (118.0, 146.0)
- moved C15 83.2 mm to (162.0, 146.0)
- moved C16 83.2 mm to (147.0, 146.0)
- moved R20 83.2 mm to (124.0, 146.0)
- moved RV7 82.8 mm to (67.0, 156.0)
- moved C11 76.5 mm to (150.0, 132.0)
- moved C12 76.5 mm to (194.0, 132.0)
- moved C13 76.5 mm to (179.0, 132.0)
- moved R17 76.5 mm to (156.0, 132.0)
- moved RV3 76.5 mm to (145.0, 137.0)
- moved RV5 72.0 mm to (160.0, 137.0)
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Routing:
- net GND: track 390.8 -> 485.9 mm
- net Net-(RV11-Pad3): track 0.00 -> 78.9 mm
- net /fx_return: track 0.00 -> 69.5 mm
- net /post_stage_1: track 0.00 -> 68.0 mm
- net Net-(C15-Pad1): track 15.0 -> 69.8 mm
- net Net-(RV3-Pad2): track 0.00 -> 52.9 mm
- net Net-(R22-Pad2): track 0.00 -> 39.4 mm
- net Net-(C14-Pad2): track 0.00 -> 33.6 mm
- net Net-(R8-Pad2): track 0.00 -> 33.5 mm
- net Net-(C11-Pad2): track 68.1 -> 38.2 mm
- net Net-(R19-Pad2): track 0.00 -> 23.5 mm
- net Net-(C5-Pad1): track 0.00 -> 20.8 mm
- net Net-(C13-Pad1): track 0.00 -> 18.8 mm
- net Net-(C12-Pad1): track 0.00 -> 17.5 mm
- net Net-(RV10-Pad3): track 0.00 -> 14.0 mm
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
Commit message: genug fuer heute
Parts:
- moved D6 80.1 mm to (218.0, 148.0), turned to 90 degrees
- moved R21 75.0 mm to (201.0, 144.5), turned to 90 degrees
- moved R22 73.8 mm to (210.0, 148.0), turned to 90 degrees
- moved D5 64.0 mm to (193.0, 142.0), turned to 270 degrees
Routing:
- net /HV_in: track 32.8 -> 216.2 mm
- net GND: track 485.9 -> 641.4 mm
- net /fx_send: track 82.1 -> 168.7 mm
- net /12V: track 63.6 -> 140.4 mm
- net Net-(R22-Pad2): track 39.4 -> 93.3 mm
- net Net-(C12-Pad1): track 17.5 -> 55.4 mm
- net Net-(C11-Pad2): track 38.2 -> 15.1 mm
- net Net-(R21-Pad2): track 0.00 -> 16.4 mm
- net /HV_A: track 125.3 -> 122.3 mm

Commit message: new evening
Routing:
- net Net-(R22-Pad2): track 93.3 -> 29.4 mm
- net GND: track 641.4 -> 688.7 mm
- net /12V: track 140.4 -> 177.6 mm
- net Net-(R21-Pad2): track 16.4 -> 13.6 mm
Changed lines of the file:
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@@
     (thickness 1.6)
     (drawings 11)
-    (tracks 459)
+    (tracks 462)
     (zones 0)
     (modules 83)
@@
   (segment (start 183 126) (end 168.99254 126) (width 1) (layer F.Cu) (net 2))
   (segment (start 54 140) (end 49 140) (width 1) (layer F.Cu) (net 2))
+  (segment (start 240.75 128.65) (end 240.2 129.2) (width 1) (layer B.Cu) (net 2))
+  (segment (start 240.75 105.99) (end 240.75 128.65) (width 1) (layer B.Cu) (net 2))
+  (segment (start 240.2 130.5) (end 240.2 129.2) (width 1) (layer B.Cu) (net 2))
+  (segment (start 191 140) (end 193 142) (width 1) (layer F.Cu) (net 2))
+  (segment (start 191 137) (end 191 140) (width 1) (layer F.Cu) (net 2))
+  (segment (start 192.579998 142) (end 193 142) (width 1) (layer B.Cu) (net 2))
+  (segment (start 187 147.579998) (end 192.579998 142) (width 1) (layer B.Cu) (net 2))
+  (segment (start 187 156) (end 187 147.579998) (width 1) (layer B.Cu) (net 2))
   (segment (start 34 117) (end 35 116) (width 1) (layer B.Cu) (net 5))
   (segment (start 30 117) (end 34 117) (width 1) (layer B.Cu) (net 5))
@@
   (segment (start 144.400001 130.099999) (end 154.099999 130.099999) (width 1) (layer B.Cu) (net 13))
   (segment (start 142.5 132) (end 144.400001 130.099999) (width 1) (layer B.Cu) (net 13))
-  (segment (start 181.08 137) (end 186 137) (width 1) (layer B.Cu) (net 14))
-  (segment (start 191 132) (end 194 132) (width 1) (layer B.Cu) (net 14))
-  (segment (start 186 137) (end 191 132) (width 1) (layer B.Cu) (net 14))
   (segment (start 178.54 137) (end 181.08 137) (width 1) (layer B.Cu) (net 14))
   (segment (start 145 137) (end 145 139) (width 1) (layer F.Cu) (net 14))
@@
   (segment (start 176.742081 140) (end 178.54 138.202081) (width 1) (layer F.Cu) (net 14))
   (segment (start 146 140) (end 176.742081 140) (width 1) (layer F.Cu) (net 14))
+  (segment (start 190 132) (end 194 132) (width 1) (layer B.Cu) (net 14))
+  (segment (start 186.950001 135.049999) (end 190 132) (width 1) (layer B.Cu) (net 14))
+  (segment (start 181.08 137) (end 183.030001 135.049999) (width 1) (layer B.Cu) (net 14))
+  (segment (start 183.030001 135.049999) (end 186.950001 135.049999) (width 1) (layer B.Cu) (net 14))
   (segment (start 173.400001 130.099999) (end 171.5 132) (width 1) (layer B.Cu) (net 15))
   (segment (start 184.599999 130.099999) (end 173.400001 130.099999) (width 1) (layer B.Cu) (net 15))
@@
   (segment (start 72 139.54) (end 77 134.54) (width 1) (layer F.Cu) (net 39))
   (segment (start 72 156) (end 72 139.54) (width 1) (layer F.Cu) (net 39))
-  (segment (start 201 142) (end 201 136) (width 1) (layer B.Cu) (net 40))
-  (segment (start 201 136) (end 199 134) (width 1) (layer B.Cu) (net 40))
-  (segment (start 199 134) (end 195 134) (width 1) (layer B.Cu) (net 40))
-  (segment (start 193.54 135.46) (end 193.54 137) (width 1) (layer B.Cu) (net 40))
-  (segment (start 195 134) (end 193.54 135.46) (width 1) (layer B.Cu) (net 40))
-  (segment (start 179 143) (end 158 143) (width 1) (layer B.Cu) (net 41))
-  (segment (start 153 143) (end 151 143) (width 1) (layer B.Cu) (net 41))
-  (segment (start 158 143) (end 153 143) (width 1) (layer B.Cu) (net 41))
-  (segment (start 142 141) (end 140.599999 139.599999) (width 1) (layer B.Cu) (net 41))
-  (segment (start 148 141) (end 142 141) (width 1) (layer B.Cu) (net 41))
-  (segment (start 150 143) (end 148 141) (width 1) (layer B.Cu) (net 41))
-  (segment (start 153 143) (end 150 143) (width 1) (layer B.Cu) (net 41))
-  (segment (start 187 151) (end 186.5 150.5) (width 1) (layer B.Cu) (net 41))
-  (segment (start 192 156) (end 186.5 150.5) (width 1) (layer B.Cu) (net 41))
-  (segment (start 186.5 150.5) (end 179 143) (width 1) (layer B.Cu) (net 41))
+  (segment (start 201 139.033998) (end 201 142) (width 1) (layer B.Cu) (net 40))
+  (segment (start 194.28792 135.049999) (end 197.016001 135.049999) (width 1) (layer B.Cu) (net 40))
+  (segment (start 193.54 135.797919) (end 194.28792 135.049999) (width 1) (layer B.Cu) (net 40))
+  (segment (start 197.016001 135.049999) (end 201 139.033998) (width 1) (layer B.Cu) (net 40))
+  (segment (start 193.54 137) (end 193.54 135.797919) (width 1) (layer B.Cu) (net 40))
   (segment (start 210 145.46) (end 212.46 145.46) (width 1) (layer B.Cu) (net 41))
-  (segment (start 209.812002 151) (end 187 151) (width 1) (layer B.Cu) (net 41))
   (segment (start 212.46 145.46) (end 213 146) (width 1) (layer B.Cu) (net 41))
   (segment (start 213 146) (end 213 147.812002) (width 1) (layer B.Cu) (net 41))
   (segment (start 213 147.812002) (end 209.812002 151) (width 1) (layer B.Cu) (net 41))
+  (segment (start 192 156) (end 197 151) (width 1) (layer B.Cu) (net 41))
+  (segment (start 209.812002 151) (end 197 151) (width 1) (layer B.Cu) (net 41))
   (segment (start 113 137) (end 124 137) (width 1) (layer B.Cu) (net 42))
   (segment (start 57.87756 104.9101) (end 61 101.78766) (width 1) (layer B.Cu) (net 43))
@@
   (segment (start 203.5 118.25) (end 193.75 128) (width 1) (layer F.Cu) (net 50))
   (segment (start 193.75 128) (end 163.347998 128) (width 1) (layer F.Cu) (net 50))
-  (segment (start 151 141) (end 147.54 137.54) (width 1) (layer B.Cu) (net 51))
+  (segment (start 235.67 105.99) (end 223.66 118) (width 1) (layer F.Cu) (net 50))
+  (segment (start 203.75 118) (end 203.5 118.25) (width 1) (layer F.Cu) (net 50))
+  (segment (start 223.66 118) (end 203.75 118) (width 1) (layer F.Cu) (net 50))
   (segment (start 147.54 137.54) (end 147.54 137) (width 1) (layer B.Cu) (net 51))
-  (segment (start 196.08 137) (end 196.08 138.202081) (width 1) (layer B.Cu) (net 51))
   (segment (start 196.08 138.202081) (end 195.282081 139) (width 1) (layer B.Cu) (net 51))
-  (segment (start 195.282081 139) (end 187 139) (width 1) (layer B.Cu) (net 51))
-  (segment (start 187 139) (end 185 141) (width 1) (layer B.Cu) (net 51))
-  (segment (start 185 141) (end 151 141) (width 1) (layer B.Cu) (net 51))
+  (segment (start 196.08 137) (end 196.08 138.202081) (width 1) (layer B.Cu) (net 51))
+  (segment (start 195.282081 139) (end 190 139) (width 1) (layer B.Cu) (net 51))
+  (segment (start 151 141) (end 147.54 137.54) (width 1) (layer B.Cu) (net 51))
+  (segment (start 190 139) (end 188 141) (width 1) (layer B.Cu) (net 51))
+  (segment (start 188 141) (end 151 141) (width 1) (layer B.Cu) (net 51))
   (segment (start 165.08 137) (end 176 137) (width 1) (layer B.Cu) (net 52))
   (segment (start 194.729999 153.729999) (end 197 156) (width 1) (layer F.Cu) (net 53))

Commit message: snap
Parts:
- moved D2 29.9 mm to (56.9, 144.6)
- moved R18 24.0 mm to (81.9, 134.6)
- moved RV2 16.3 mm to (88.0, 151.0)
- moved D3 16.0 mm to (89.5, 141.0)
- moved R19 11.2 mm to (81.9, 142.1)
- moved RV1 11.2 mm to (52.0, 151.0)
- moved D1 8.62 mm to (56.9, 137.2), turned to 90 degrees
- moved R23 4.42 mm to (114.9, 141.0)
Routing:
- net GND: track 688.7 -> 639.2 mm
- net Net-(R18-Pad2): track 6.06 -> 37.5 mm
- net Net-(C5-Pad1): track 20.8 -> 35.2 mm
- net Net-(C3-Pad2): track 21.6 -> 33.5 mm
- net /post_stage_1: track 68.0 -> 78.6 mm
- net /clean_channel_bypass: track 111.9 -> 122.1 mm
- net Net-(R19-Pad2): track 23.5 -> 15.5 mm
- net Net-(R8-Pad2): track 33.5 -> 31.7 mm
- net /od_A: track 50.7 -> 52.5 mm
