File: 6N2P_amp.sch (KiCad schematic (older format))
At the start: 91 parts, among them J1 guitar_in, J2 speaker, J3 fx_send, J4 fx_return, J5 foot_sw, U1 ECC83, U2 ECC83, U3 6N1P, U4 DSN-MINI-360, U5 DSN-MINI-360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

Commit message: resistors and spacings
Other:
- note added: "TODO:\n\nfootswitch -> 2n7000 inverter to swith CL and OD nets\npower input hohlstecker pcb\n\n"
- note removed: "TODO:\n\nfootswitch -> 2n7000 inverter to swith CL and OD nets\npower input hohlstecker pcb\n\n470R resistors for LEDs\n25mm space between LDR and LED"
Changed lines of the file:
@@
 	12900 8500 12900 8450
 Text Notes 1550 13600 0    118  ~ 0
-TODO:\n\nfootswitch -> 2n7000 inverter to swith CL and OD nets\npower input hohlstecker pcb\n\n470R resistors for LEDs\n25mm space between LDR and LED
+TODO:\n\nfootswitch -> 2n7000 inverter to swith CL and OD nets\npower input hohlstecker pcb\n\n
 $Comp
 L micha_custom:6.3MMTRSSwitched J5
